File: SCT3811.kicad_sch (KiCad schematic)
At the start: 64 parts, among them U1 MMZ1005B601CT000, U2 MMZ1005B601CT000, U23 CMX994E1, U39 MMZ1005B601CT000, X2 26MHz

Commit message: sec
Parts:
- L46: footprint (none) -> easyeda2kicad_foorprint:L0402
Changed lines of the file:
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@@
 			)
 		)
-		(property "Footprint" ""
+		(property "Footprint" "easyeda2kicad_foorprint:L0402"
 			(at 52.07 119.38 0)
 			(effects
